Commit message: get urdf of parametric 1dof rock

File: onshape/rock1.urdf (robot description, URDF)
Before this commit: robot test, 3 links, 2 joints
Links:
- removed link hammer_1
- removed link mount_1
- removed link root_1
- added link Part_2_1, mass 0; collision mesh filename=meshes/Part_2_1.stl; visual mesh filename=meshes/Part_2_1.stl
- added link Part_3_1, mass 0; collision mesh filename=meshes/Part_3_1.stl; visual mesh filename=meshes/Part_3_1.stl
- added link Part_4_1, mass 0; collision mesh filename=meshes/Part_4_1.stl; visual mesh filename=meshes/Part_4_1.stl
- added link foot_1, mass 0; collision mesh filename=meshes/foot_1.stl; visual mesh filename=meshes/foot_1.stl
Joints:
- added joint Slider_1: type prismatic, parent Part_2_1, child Part_3_1, origin xyz=0.0094664182 -0.011587739 -2.7572687e-19 rpy=-1.5707963 0 -0.78539816, axis 0 0 -1, limit lower=-0.1 upper=0.1 effort=1 velocity=1
- joint Revolute_1: child hammer_1 -> Part_2_1; origin xyz=-0.005 0.06045085 -0.01 rpy=-3.1415927 1.5707963 0 -> xyz=-2.1684043e-19 0 0.0015 rpy=-1.5707963 0 0; parent mount_1 -> foot_1
- joint Revolute_2: child mount_1 -> Part_4_1; origin xyz=2.1906919e-16 -0.010032667 -0.053219852 rpy=1.5707963 0 -9.9920072e-16 -> xyz=-0.001 -4.1359031e-19 -0.002 rpy=0 0 0; parent root_1 -> Part_3_1
