Commit message: a bunch of training, parameter tuning

File: onshape/pmrock/pmrock.urdf (robot description, URDF)
Before this commit: robot pmrock, 3 links, 2 joints
Links:
- link foot_1: mass 0.0014241887 -> 0.011393509
- link pendulum_1: mass 0.0998712 -> 0.150; geometry visual mesh filename=meshes/pendulum_1.stl
- link shell_com_1: mass 0 -> 0.100; geometry visual mesh filename=meshes/shell_com_1.stl
Joints:
- joint Fastened_1: origin xyz=0.002 0 0.076 rpy=3.1415927 0 0 -> xyz=0.002 0 0.115 rpy=3.1415927 0 0
