Commit message: figure out how to set initial dof and base vels

File: onshape/balo/balo.urdf (robot description, URDF)
Before this commit: robot balo, 3 links, 2 joints
Links:
- removed link bottomshell_1
- removed link topshell_1
- added link shell_1, mass 0.088985938; collision mesh filename=meshes/shell_1.stl; visual mesh filename=meshes/shell_1.stl
- link pendulum_1: mass 0 -> 0.025374834; geometry visual mesh filename=meshes/pendulum_1.stl
Joints:
- removed joint Fastened_2
- joint Revolute_1: origin xyz=-1.9306432e-07 -0.02472204 -0.021835193 rpy=-2.2455373 0 0 -> xyz=1.022949e-05 -1.6753779e-06 9.9866003e-06 rpy=3.1415927 0 0; parent bottomshell_1 -> shell_1
